File: receiver/receiver/receiver.sch (KiCad schematic (older format))
At the start: 3 parts

Commit message: add 100mF capacitor
Parts:
- C1: renamed from C?; value CP -> 100microF; footprint (none) -> Capacitor_THT:CP_Radial_D4.0mm_P2.00mm
Changed lines of the file:
@@
 F 0 "#PWR02" H 4950 1150 50  0001 C CNN
 F 1 "+7.5V" H 4965 1473 50  0000 C CNN
-F 2 "" H 4950 1300 50  0001 C CNN
+F 2 "Connector_PinHeader_2.54mm:PinHeader_1x01_P2.54mm_Vertical" H 4950 1300 50  0001 C CNN
 F 3 "" H 4950 1300 50  0001 C CNN
 	1    4950 1300
@@
 F 0 "#PWR03" H 5450 1050 50  0001 C CNN
 F 1 "GND" H 5455 1127 50  0000 C CNN
-F 2 "" H 5450 1300 50  0001 C CNN
+F 2 "Connector_PinHeader_2.54mm:PinHeader_1x01_P2.54mm_Vertical" H 5450 1300 50  0001 C CNN
 F 3 "" H 5450 1300 50  0001 C CNN
 	1    5450 1300
@@
 	7550 2700 7750 2700
 $Comp
-L Device:CP C?
+L Device:CP C1
 U 1 1 5F24AE15
 P 7200 2250
-F 0 "C?" V 6945 2250 50  0000 C CNN
-F 1 "CP" V 7050 2250 50  0000 C CNN
-F 2 "" H 7238 2100 50  0001 C CNN
+F 0 "C1" V 6945 2250 50  0000 C CNN
+F 1 "100microF" V 7050 2250 50  0000 C CNN
+F 2 "Capacitor_THT:CP_Radial_D4.0mm_P2.00mm" H 7238 2100 50  0001 C CNN
 F 3 "~" H 7200 2250 50  0001 C CNN
 	1    7200 2250

Commit message: add pins
Parts:
- added C2: 470microF, Capacitor_THT:CP_Radial_D8.0mm_P3.50mm, symbol Device:C
- added C3: 0.1microF, Capacitor_THT:C_Disc_D3.0mm_W2.0mm_P2.50mm, symbol Device:CP
- added C4: 470microF, Capacitor_THT:CP_Radial_D8.0mm_P3.50mm, symbol Device:CP
- added C5, C6: 0.1microF, Capacitor_THT:C_Disc_D3.0mm_W2.0mm_P2.50mm, symbol Device:C
- added D3, D4, D5, D6: servo_connector, Connector_PinHeader_2.54mm:PinHeader_1x03_P2.54mm_Vertical, symbol pinconnectors:servo_connector
Connections:
- net +3V3: now also C6.1
- net +7.5V: now also C2.2, C3.2, C4.2, C5.2, D3.2 (VCC), D4.2 (VCC), D5.2 (VCC), D6.2 (VCC)
- net GND: now also C2.1, C3.1, C4.1, C5.1, D3.1 (GND), D4.1 (GND), D5.1 (GND), D6.1 (GND)
- net GND1: now also C6.2
- net D5: now reaches D1.10 (D5)
- net D5: now also D3.3 (PWM)
- net D21: now reaches D1.14 (D21)
- net D21: now also D4.3 (PWM)
- net D22: now reaches D1.17 (D22)
- net D22: now also D5.3 (PWM)
- net D23: now reaches D1.18 (D23)
- net D23: now also D6.3 (PWM)
Other:
- moved on the sheet: C1, D1, D2

Commit message: LM2596
Parts:
- added D10: cleat_2pin, common:cleat_2pin, symbol common:cleat_2pin
- added D11: LM2596, common:LM2596, symbol common:LM2596
- added D7: 3.3V, common:3.3V-converter, symbol common:3.3V
- added D8: 5.0V, common:5.0V-converter, symbol common:5.0V
- added D9: nextion, symbol common:nextion
Connections:
- net +7.5V: now also D11.4 (OUT+), D7.1 (IN), D8.1 (IN)
- net GND: now also D10.2 (MINUS), D11.2 (-IN); no longer C2.1, C3.1, C4.1, C5.1, D1.33 (GND), D3.1 (GND), D4.1 (GND), D5.1 (GND), D6.1 (GND)
- net GND1: now also C2.1, C3.1, C4.1, C5.1, D1.33 (GND), D3.1 (GND), D4.1 (GND), D5.1 (GND), D6.1 (GND), D11.3 (OUT-), D7.2 (GND), D8.2 (GND), D9.4 (GND); no longer C1.2, C6.2, D1.19 (GND), D2.1 (GND), D2.5 (IRQ)
- net at D1.15 (RX): now also D9.3 (RX)
- net at D1.16 (TX): now also D9.2 (TX)
- new net +12V: D10.1 (PLUS), D11.1 (+IN)
- new net +5V: D8.3 (OUT), D9.1 (+5V)
- new net GND2: C1.2, C6.2, D1.19 (GND), D2.1 (GND), D2.5 (IRQ)
